File: rev_b/hdw/Nixie_Clock_Core/USB_Telemetry.kicad_sch (KiCad schematic)
At the start: 7 parts, among them U2601 INA219BxDCN

Commit message: lots of rev B control board schematic progress
Parts:
- renumbered U2601 to U?
