File: rev_b/hdw/Nixie_Clock_Core/Nixie_Clock_Core.kicad_pcb (KiCad board)
At the start: 6 copper layers, 200 x 50 mm, 325 parts, among them J1301 USB_B_Mini, J1901 Conn_02x32_Odd_Even, J201 +24V IN, J2101 I2C, J2102 USB UART, J801 PICKIT4, Q2101 BSS214NW, Q401 BSS214NW, Q402 ZXMS6004FFTA, Q601 IRFL214, Q701 BSS192PH6327FTSA1, Q801 BSS214NW, SW801 MRST, U1001 PIC32MZ2048EFG100_IPF, U1101 74LVC1G97, U1201 DS3231MZ, U1202 TLV6700, U1301 TLV6700, U1302 FT234XD, U1303 74LVC1G97, U1304 ISO7321C, U1305 TPD3S014DBVR, U1401 DS1683, U1501 74LVC1G97, U1502 74LVC1G97, U1503 74LVC1G97, U1504 74LVC1G97, U1505 74LVC1G97, U1601 74LVC1G97, U1602 74LVC1G97, U1603 74LVC1G97, U1604 74LVC1G97, U1701 74VHC541, U1702 74VHC541, U1703 74VHC541, U1801 TCA9803, U1802 74VHC541, U201 TPS26600RHFT, U2101 LTC6900, U2102 74LVC1G97, U2103 MCP9804, U301 INA219BxDCN, U302 MCP9804, U401 LT8609A-DD, U501 INA219BxDCN, U502 MCP9804, U601 TLV6700, U602 LT3757, U603 TLV6700, U701 OPA333xxDCK, U702 MCP9804, U703 INA219BxDCN, U704 OPA333xxDCK, U705 OPA333xxDCK, X1101 ASE-8.000MHz, X1102 ECS-327KE

Commit message: hid all passive refdes on core PCB
Parts:
- moved C301 203.6 mm to (419.2, 27.6)
- moved C302 203.6 mm to (419.2, 30.0)
- moved C303 203.6 mm to (419.2, 32.4)
- moved U301 203.6 mm to (423.8, 32.4)
- moved U302 203.6 mm to (423.8, 28.3)

Commit message: started grouping MCU components on PCB
Parts:
- C1101, C801, D801, Q801, R801, R802, R803, R804, R805: moved to B.Cu
- moved L1101 293.2 mm to (309.3, 298.7), turned to 90 degrees
- moved C1102 290.0 mm to (307.0, 297.9), turned to 180 degrees
- moved U1101 288.2 mm to (306.6, 288.7), turned to -90 degrees
- moved C1104 287.2 mm to (307.0, 299.3), turned to 180 degrees
- moved X1101 287.0 mm to (307.0, 295.4), turned to 180 degrees
- moved R1103 286.0 mm to (302.7, 295.4), turned to 90 degrees
- moved C1101 284.5 mm to (306.6, 288.7), turned to 90 degrees
- moved R1102 282.3 mm to (306.6, 291.2)
- moved R1105 281.0 mm to (304.2, 295.4), turned to 90 degrees
- moved TP1101 271.1 mm to (309.2, 278.5)
- moved R1101 270.3 mm to (309.2, 276.0), turned to 90 degrees
- moved L1102 267.6 mm to (310.0, 270.7), turned to 180 degrees
- moved R1104 266.8 mm to (306.6, 277.3), turned to 180 degrees
- moved C1103 266.1 mm to (309.2, 272.9), turned to -90 degrees
- moved X1102 265.6 mm to (306.6, 272.9), turned to -90 degrees
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Connections:
- R1105 pad 1: PIC32MZ_POSC_EC -> Net-(X1101-OUT)
- R1106 pad 1: PIC32MZ_SOSC_EC -> Net-(X1102-OUT)
Other:
- board text added: "REFCLK1"

Commit message: much more component placement on core board
Parts:
- removed R1804: 10K, Resistors_SMD:R_0603
- C1802, C1803, C1804, C1805, R1701, R1702, R1703, R1801, R1802, R1806, RN1701, RN1702, RN1703, RN1801, RN1802: moved to B.Cu
- moved C1802 288.2 mm to (385.5, 313.8), turned to -90 degrees
- moved C1804 283.7 mm to (390.5, 313.8), turned to -90 degrees
- moved C1803 283.2 mm to (387.1, 313.8), turned to -90 degrees
- moved R1803 282.1 mm to (392.3, 315.0), turned to 90 degrees
- moved R1801 281.6 mm to (389.5, 308.2), turned to 180 degrees
- moved U1802 281.1 mm to (388.0, 304.6)
- moved U1801 280.2 mm to (388.0, 313.8)
- moved C1805 279.9 mm to (388.9, 313.8), turned to -90 degrees
- moved RN1802 278.7 mm to (386.3, 304.6), turned to 180 degrees
- moved C1801 277.7 mm to (388.0, 300.9), turned to 180 degrees
- moved RN1801 275.4 mm to (389.5, 305.1)
- moved R1805 275.3 mm to (392.3, 312.4), turned to -90 degrees
- moved R1802 274.3 mm to (388.0, 301.6), turned to 180 degrees
- moved R1806 271.8 mm to (386.3, 307.7), turned to 180 degrees
- moved U1401 260.6 mm to (440.1, 290.8)
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Connections:
- RN1801 pad 10: Pushbutton_6 -> Pushbutton_1
- RN1801 pad 11: Pushbutton_5 -> Pushbutton_2
- RN1801 pad 12: Pushbutton_4 -> Pushbutton_3
- RN1801 pad 13: Pushbutton_3 -> Pushbutton_4
- RN1801 pad 14: Pushbutton_2 -> Pushbutton_5
- RN1801 pad 15: Pushbutton_1 -> Pushbutton_6
- RN1801 pad 16: Pushbutton_0 -> unconnected-(RN1801-R1.2-Pad16)
- RN1801 pad 9: unconnected-(RN1801-R8.2-Pad9) -> Pushbutton_0

Commit message: arranged USB components on PCB, added USB isolator Bypass
Parts:
- removed D201: 48V, Diodes_SMD:D_SMA
- added C1310: 0.1uF, Capacitors_SMD:C_0603, B.Cu at (369.6, 398.9)
- added C1311: 10uF, Capacitors_SMD:C_0603, B.Cu at (369.6, 397.5)
- added C1312: 0.1uF, Capacitors_SMD:C_0603, B.Cu at (369.6, 403.8)
- added C1313: 10uF, Capacitors_SMD:C_0603, B.Cu at (369.6, 405.2)
- C1202, C1203, C1204, C1205, C1301, C1302, C1303, C1304, C1305, C1306, C1307, C1308, C1309, C202, C205, C206, C2102, C301, C302, C303, D2101, L1301, L1302, R1201, R1203, R1308, R1309, R201, R202, R203, R207, R210, R2104, R2107, R211, R2111, U1302, U1303, U301, U302: moved to B.Cu
- moved C1202 365.5 mm to (389.6, 373.8), turned to -90 degrees
- moved R1201 365.5 mm to (372.8, 373.6), turned to 180 degrees
- moved U1201 363.5 mm to (385.8, 372.5)
- moved C1203 363.1 mm to (388.2, 373.8), turned to -90 degrees
- moved R1202 363.0 mm to (372.8, 373.6)
- moved U1202 361.7 mm to (372.8, 371.0)
- moved C1204 359.2 mm to (385.8, 372.5)
- moved BT1202 358.8 mm to (379.6, 356.5)
- moved TP1201 357.0 mm to (378.6, 370.0)
- moved R1203 356.5 mm to (372.8, 369.5), turned to 180 degrees
- moved C1205 354.2 mm to (372.8, 371.0), turned to 180 degrees
- moved C207 342.1 mm to (307.6, 321.8), turned to -90 degrees
- moved TP202 342.0 mm to (296.8, 327.2)
- moved J201 341.6 mm to (291.8, 320.6)
- moved C201 337.2 mm to (294.4, 325.2), turned to -90 degrees
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Other:
- board text added: "+24V"
- board text added: "+24Vin"
- board text added: "+5V USB"
- board text added: "+5V USB PGOOD"
- board text added: "USB LINK"

Commit message: much more core board component plcement
Parts:
- C1501, C1502, C1503, C1504, C1505, C1601, C1602, C1603, C1604, R1501, R1601, R1602, R1605, R1606: moved to B.Cu
- moved D1503 275.7 mm to (429.2, 292.1)
- moved C1503 274.7 mm to (426.0, 291.4), turned to 180 degrees
- moved C1604 273.0 mm to (424.1, 260.5), turned to 180 degrees
- moved C1603 271.5 mm to (424.1, 256.4), turned to 180 degrees
- moved C1602 270.0 mm to (424.1, 252.2), turned to 180 degrees
- moved C1601 268.5 mm to (424.1, 248.1), turned to 180 degrees
- moved D1505 268.3 mm to (429.2, 287.9)
- moved R1504 268.0 mm to (429.2, 290.7)
- moved U1503 267.4 mm to (426.0, 291.4)
- moved C1505 267.3 mm to (426.0, 287.2), turned to 180 degrees
- moved D1502 267.2 mm to (429.2, 279.5)
- moved D1504 266.8 mm to (429.2, 283.7)
- moved U1604 266.3 mm to (424.1, 260.5)
- moved C1502 266.2 mm to (426.0, 278.8), turned to 180 degrees
- moved U1603 266.1 mm to (424.1, 256.4)
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Other:
- board text added: "+180V PGOOD"
- board text added: "+24V PGOOD"
- board text added: "+3.3V PGOOD"
- board text added: "+90V PGOOD"
- board text added: "CPU Trap"
- board text added: "Error"
- board text added: "HRTBT"
- board text added: "LOW BAT"
- board text added: "Reset"

Commit message: more core board component placement
Parts:
- added C614: 0.1uF, Capacitors_SMD:C_0603, F.Cu at (413.3, 51.2)
- C501, C502, C503, C605, C610, C611, C612, C701, C702, C703, C704, D701, Q601, R401, R611, R615, R617, R701, R702, U501, U502, U701, U702, U703: moved to B.Cu
- R610: footprint Resistors_SMD:R_0402 -> Resistors_SMD:R_0603
- moved C404 287.1 mm to (256.0, 276.6)
- moved U502 285.0 mm to (251.7, 274.5), turned to -90 degrees
- moved C409 282.4 mm to (253.5, 278.0), turned to 90 degrees
- moved R403 282.4 mm to (247.4, 276.9), turned to 180 degrees
- moved C503 282.4 mm to (251.7, 277.4)
- moved C406 281.0 mm to (248.8, 272.7), turned to -90 degrees
- moved R402 280.8 mm to (256.0, 275.1), turned to 180 degrees
- moved C401 280.6 mm to (257.6, 272.0), turned to 90 degrees
- moved R406 279.3 mm to (245.2, 265.0), turned to 90 degrees
- moved TP401 278.6 mm to (245.2, 262.1)
- moved C403 278.2 mm to (255.3, 272.0), turned to 90 degrees
- moved C501 275.6 mm to (250.6, 265.1), turned to 90 degrees
- moved C407 274.6 mm to (250.4, 270.0)
- moved L401 274.2 mm to (245.2, 270.5), turned to 90 degrees
- moved C405 274.1 mm to (258.9, 266.2), turned to 90 degrees
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Connections:
- R608 pad 1: +180V -> +90V
Other:
- board text added: "+3.3V"

Commit message: chose new IO connector, fixed some net connectivity issues
Parts:
- C1903: moved to B.Cu
- J1901: value Conn_02x32_Odd_Even -> Conn_02x32_Top_Bottom; footprint Connector_PinSocket_2.54mm:PinSocket_2x32_P2.54mm_Vertical_SMD -> Custom Footprints Library:CONN_5120527-1_TYC
- moved H2007 149.0 mm to (232.0, 71.8)
- moved H2008 133.8 mm to (232.0, 115.8)
- moved C1903 118.4 mm to (231.2, 107.8)
- moved C1902 107.2 mm to (218.9, 73.0), turned to 90 degrees
- moved C1901 106.7 mm to (224.8, 73.0), turned to 90 degrees
- moved H2005 105.1 mm to (168.4, 71.8)
- moved H2002 95.4 mm to (38.0, 71.8)
- moved H2006 82.1 mm to (168.4, 115.8)
- moved H2003 78.1 mm to (101.7, 71.8)
- moved J1901 76.3 mm to (229.4, 78.3), turned to -90 degrees
- moved H2001 55.0 mm to (38.0, 115.8)
- moved H2004 42.5 mm to (101.7, 115.8)
- moved TP601 36.1 mm to (446.9, 53.5)
- moved TP602 36.1 mm to (446.9, 56.7)
Connections:
- C1901 pad 1: +90V -> +180V
- J1901 pad 11: GND -> Cathode_0_DSP
- J1901 pad 12: GND -> Cathode_2_DSP
- J1901 pad 13: Anode_0_DSP -> Cathode_4_DSP
- J1901 pad 14: Anode_1_DSP -> Cathode_6_DSP
- J1901 pad 15: Anode_2_DSP -> Cathode_8_DSP
- J1901 pad 16: Anode_3_DSP -> Cathode_DP_DSP
- J1901 pad 17: Anode_4_DSP -> GND
- J1901 pad 18: Anode_5_DSP -> Colon_0_DSP
- J1901 pad 19: GND -> Colon_2_DSP
- J1901 pad 2: GND -> +180V
- J1901 pad 21: Cathode_0_DSP -> Pushbutton_0_DSP
- J1901 pad 22: Cathode_1_DSP -> Pushbutton_2_DSP
- J1901 pad 23: Cathode_2_DSP -> Pushbutton_4_DSP
- J1901 pad 24: Cathode_3_DSP -> Pushbutton_6_DSP
- J1901 pad 25: Cathode_4_DSP -> ~{Display_Detect_DSP}
- J1901 pad 26: Cathode_5_DSP -> I2C_DSP_SCL
- J1901 pad 27: Cathode_6_DSP -> USB_UART_TX
- J1901 pad 28: Cathode_7_DSP -> unconnected-(J1901-Pin_28-Pad28)
- J1901 pad 29: Cathode_8_DSP -> +3.3V
- J1901 pad 3: +180V -> unconnected-(J1901-Pin_3-Pad3)
- J1901 pad 30: Cathode_9_DSP -> +3.3V
- J1901 pad 31: Cathode_DP_DSP -> +3.3V
- J1901 pad 32: GND -> +3.3V
- J1901 pad 35: Colon_0_DSP -> GND
- J1901 pad 36: Colon_1_DSP -> GND
- J1901 pad 37: Colon_2_DSP -> GND
- J1901 pad 38: Colon_3_DSP -> GND
- J1901 pad 39: GND -> Anode_1_DSP
- J1901 pad 4: GND -> +90V
- J1901 pad 40: GND -> Anode_3_DSP
- J1901 pad 41: Pushbutton_0_DSP -> Anode_5_DSP
- J1901 pad 42: Pushbutton_1_DSP -> GND
- J1901 pad 43: Pushbutton_2_DSP -> Cathode_1_DSP
- J1901 pad 44: Pushbutton_3_DSP -> Cathode_3_DSP
- J1901 pad 45: Pushbutton_4_DSP -> Cathode_5_DSP
- J1901 pad 46: Pushbutton_5_DSP -> Cathode_7_DSP
- J1901 pad 47: Pushbutton_6_DSP -> Cathode_9_DSP
- J1901 pad 49: ~{Display_Detect_DSP} -> GND
- J1901 pad 5: unconnected-(J1901-Pin_5-Pad5) -> +90V
- J1901 pad 50: GND -> Colon_1_DSP
- J1901 pad 51: I2C_DSP_SCL -> Colon_3_DSP
- J1901 pad 52: I2C_DSP_SDA -> GND
- J1901 pad 53: USB_UART_TX -> Pushbutton_1_DSP
- J1901 pad 54: USB_UART_RX -> Pushbutton_3_DSP
- J1901 pad 55: unconnected-(J1901-Pin_55-Pad55) -> Pushbutton_5_DSP
- J1901 pad 56: unconnected-(J1901-Pin_56-Pad56) -> GND
- J1901 pad 57: +3.3V -> GND
- J1901 pad 58: GND -> I2C_DSP_SDA
- J1901 pad 59: +3.3V -> USB_UART_RX
- J1901 pad 60: GND -> unconnected-(J1901-Pin_60-Pad60)
- J1901 pad 61: +3.3V -> GND
- J1901 pad 63: +3.3V -> GND
- J1901 pad 7: +180V -> Anode_0_DSP
- J1901 pad 8: GND -> Anode_2_DSP
- J1901 pad 9: +180V -> Anode_4_DSP

Commit message: lots more PCB placement
Parts:
- added J202: +24V IN, Connectors:BARREL_JACK, F.Cu at (44.8, 85.7)
- C610, C801, Q801, R801, R802, R803, R804, R805: moved to F.Cu
- C705, C706, D401, R608, R609, R610, R612, R703, R704, R705, R706, R707, R708, U603, U704, U705: moved to B.Cu
- moved C1308 356.2 mm to (46.2, 105.8)
- moved C1309 356.2 mm to (46.2, 104.4)
- moved L1301 356.2 mm to (45.0, 100.6)
- moved R1308 356.2 mm to (46.2, 107.2)
- moved R1309 356.2 mm to (46.2, 103.0)
- moved U1305 356.2 mm to (46.0, 100.6)
- moved C1301 356.2 mm to (49.9, 108.8)
- moved C1302 356.2 mm to (50.1, 101.4)
- moved C1303 356.2 mm to (47.6, 109.6)
- moved C1304 356.2 mm to (51.5, 101.4)
- moved C1305 356.2 mm to (48.7, 101.4)
- moved C1306 356.2 mm to (54.3, 109.6)
- moved C1307 356.2 mm to (46.5, 100.6)
- moved C1310 356.2 mm to (58.6, 102.4)
- moved C1311 356.2 mm to (58.6, 101.0)
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Connections:
- R1801 pad 2: ~{Display_Detect} -> Pushbutton_0
- R1806 pad 2: ~{Display_Detect_DSP} -> Pushbutton_0_DSP
- R705 pad 1: +180V -> +90V
- RN1801 pad 10: Pushbutton_1 -> Pushbutton_6
- RN1801 pad 11: Pushbutton_2 -> Pushbutton_5
- RN1801 pad 12: Pushbutton_3 -> Pushbutton_4
- RN1801 pad 13: Pushbutton_4 -> Pushbutton_3
- RN1801 pad 14: Pushbutton_5 -> Pushbutton_2
- RN1801 pad 15: Pushbutton_6 -> Pushbutton_1
- RN1801 pad 9: Pushbutton_0 -> ~{Display_Detect}
- RN1802 pad 10: Pushbutton_6_DSP -> Pushbutton_1_DSP
- RN1802 pad 11: Pushbutton_5_DSP -> Pushbutton_2_DSP
- RN1802 pad 12: Pushbutton_4_DSP -> Pushbutton_3_DSP
- RN1802 pad 13: Pushbutton_3_DSP -> Pushbutton_4_DSP
- RN1802 pad 14: Pushbutton_2_DSP -> Pushbutton_5_DSP
- RN1802 pad 15: Pushbutton_1_DSP -> Pushbutton_6_DSP
- RN1802 pad 16: Pushbutton_0_DSP -> ~{Display_Detect_DSP}
- U1802 pad 11: ~{Display_Detect} -> Pushbutton_0
- U1802 pad 12: Pushbutton_6 -> Pushbutton_1
- U1802 pad 13: Pushbutton_5 -> Pushbutton_2
- U1802 pad 14: Pushbutton_4 -> Pushbutton_3
- U1802 pad 15: Pushbutton_3 -> Pushbutton_4
- U1802 pad 16: Pushbutton_2 -> Pushbutton_5
- U1802 pad 17: Pushbutton_1 -> Pushbutton_6
- U1802 pad 18: Pushbutton_0 -> ~{Display_Detect}
- U1802 pad 2: Pushbutton_0_DSP -> ~{Display_Detect_DSP}
- U1802 pad 3: Pushbutton_1_DSP -> Pushbutton_6_DSP
- U1802 pad 4: Pushbutton_2_DSP -> Pushbutton_5_DSP
- U1802 pad 5: Pushbutton_3_DSP -> Pushbutton_4_DSP
- U1802 pad 6: Pushbutton_4_DSP -> Pushbutton_3_DSP
- U1802 pad 7: Pushbutton_5_DSP -> Pushbutton_2_DSP
- U1802 pad 8: Pushbutton_6_DSP -> Pushbutton_1_DSP
- U1802 pad 9: ~{Display_Detect_DSP} -> Pushbutton_0_DSP
Other:
- board text added: "+180V"
- board text added: "+90V"
- board text added: "GND"
- board text added: "I2C"
- board text added: "RX"
- board text added: "SCL"
- board text added: "SDA"
- board text added: "TX"
- board text added: "USB UART"
- board text added: "VBAT"
