File: rev_b/hdw/Nixie_Clock_Core/PIC32MZ.kicad_sch (KiCad schematic)
At the start: 3 parts, among them U1002 PIC32MZ2048EFG100_IPF

Commit message: lots of rev B control board schematic progress
Parts:
- renumbered R1003 to R?, R1004 to R?, U1002 to U?
Changed lines of the file:
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@@
   (symbol (lib_id "Custom_Library:R_Custom") (at 211.328 103.632 0) (unit 1)
     (in_bom yes) (on_board yes) (dnp no)
-    (property "Reference" "R1003" (at 209.296 103.632 0)
+    (property "Reference" "R?" (at 209.296 103.632 0)
       (effects (font (size 1.27 1.27)) (justify right))
     )
@@
       (project "Nixie_Clock_Core"
         (path "/16fdce21-b570-4d81-a458-e8839d611806/f7cc5c4d-c1a6-4096-b212-cb6ae1584770"
-          (reference "R1003") (unit 1)
+          (reference "R?") (unit 1)
         )
       )
@@
         )
         (path "/22e05ee1-b227-4be7-9418-94433f274720/00000000-0000-0000-0000-00005f5829d3"
-          (reference "R1101") (unit 1)
+          (reference "R?") (unit 1)
         )
         (path "/22e05ee1-b227-4be7-9418-94433f274720/00000000-0000-0000-0000-00005c1de17a"
@@
   (symbol (lib_id "Custom_Library:+3.3VA_MZ") (at 113.03 22.352 0) (unit 1)
     (in_bom yes) (on_board yes) (dnp no)
-    (property "Reference" "#PWR01007" (at 113.03 26.162 0)
+    (property "Reference" "#PWR?" (at 113.03 26.162 0)
       (effects (font (size 1.27 1.27)) hide)
     )
@@
       (project "Nixie_Clock_Core"
         (path "/16fdce21-b570-4d81-a458-e8839d611806/f7cc5c4d-c1a6-4096-b212-cb6ae1584770"
-          (reference "#PWR01007") (unit 1)
-        )
-      )
-      (project "LED_Panel_Controller"
-        (path "/22e05ee1-b227-4be7-9418-94433f274720/00000000-0000-0000-0000-00005f5829d3"
-          (reference "#PWR01102") (unit 1)
+          (reference "#PWR?") (unit 1)
+        )
+      )
+      (project "LED_Panel_Controller"
+        (path "/22e05ee1-b227-4be7-9418-94433f274720/00000000-0000-0000-0000-00005f5829d3"
+          (reference "#PWR?") (unit 1)
         )
       )
@@
   (symbol (lib_id "Custom_Library:R_Custom") (at 226.314 103.632 0) (unit 1)
     (in_bom yes) (on_board yes) (dnp no)
-    (property "Reference" "R1004" (at 224.282 103.632 0)
+    (property "Reference" "R?" (at 224.282 103.632 0)
       (effects (font (size 1.27 1.27)) (justify right))
     )
@@
       (project "Nixie_Clock_Core"
         (path "/16fdce21-b570-4d81-a458-e8839d611806/f7cc5c4d-c1a6-4096-b212-cb6ae1584770"
-          (reference "R1004") (unit 1)
+          (reference "R?") (unit 1)
         )
       )
@@
         )
         (path "/22e05ee1-b227-4be7-9418-94433f274720/00000000-0000-0000-0000-00005f5829d3"
-          (reference "R1102") (unit 1)
+          (reference "R?") (unit 1)
         )
         (path "/22e05ee1-b227-4be7-9418-94433f274720/00000000-0000-0000-0000-00005c1de17a"
@@
   (symbol (lib_id "power:+3.3V") (at 125.73 22.352 0) (unit 1)
     (in_bom yes) (on_board yes) (dnp no)
-    (property "Reference" "#PWR01009" (at 125.73 26.162 0)
+    (property "Reference" "#PWR?" (at 125.73 26.162 0)
       (effects (font (size 1.27 1.27)) hide)
     )
@@
       (project "Nixie_Clock_Core"
         (path "/16fdce21-b570-4d81-a458-e8839d611806/f7cc5c4d-c1a6-4096-b212-cb6ae1584770"
-          (reference "#PWR01009") (unit 1)
-        )
-      )
-      (project "LED_Panel_Controller"
-        (path "/22e05ee1-b227-4be7-9418-94433f274720/00000000-0000-0000-0000-00005f5829d3"
-          (reference "#PWR01104") (unit 1)
+          (reference "#PWR?") (unit 1)
+        )
+      )
+      (project "LED_Panel_Controller"
+        (path "/22e05ee1-b227-4be7-9418-94433f274720/00000000-0000-0000-0000-00005f5829d3"
+          (reference "#PWR?") (unit 1)
         )
       )
@@
   (symbol (lib_id "power:+3.3V") (at 226.314 99.822 0) (unit 1)
     (in_bom yes) (on_board yes) (dnp no)
-    (property "Reference" "#PWR01012" (at 226.314 103.632 0)
+    (property "Reference" "#PWR?" (at 226.314 103.632 0)
       (effects (font (size 1.27 1.27)) hide)
     )
@@
       (project "Nixie_Clock_Core"
         (path "/16fdce21-b570-4d81-a458-e8839d611806/f7cc5c4d-c1a6-4096-b212-cb6ae1584770"
-          (reference "#PWR01012") (unit 1)
-        )
-      )
-      (project "LED_Panel_Controller"
-        (path "/22e05ee1-b227-4be7-9418-94433f274720/00000000-0000-0000-0000-00005f5829d3"
-          (reference "#PWR01107") (unit 1)
+          (reference "#PWR?") (unit 1)
+        )
+      )
+      (project "LED_Panel_Controller"
+        (path "/22e05ee1-b227-4be7-9418-94433f274720/00000000-0000-0000-0000-00005f5829d3"
+          (reference "#PWR?") (unit 1)
         )
       )
@@
   (symbol (lib_id "power:+3.3V") (at 211.328 99.822 0) (unit 1)
     (in_bom yes) (on_board yes) (dnp no)
-    (property "Reference" "#PWR01011" (at 211.328 103.632 0)
+    (property "Reference" "#PWR?" (at 211.328 103.632 0)
       (effects (font (size 1.27 1.27)) hide)
     )
@@
       (project "Nixie_Clock_Core"
         (path "/16fdce21-b570-4d81-a458-e8839d611806/f7cc5c4d-c1a6-4096-b212-cb6ae1584770"
-          (reference "#PWR01011") (unit 1)
-        )
-      )
-      (project "LED_Panel_Controller"
-        (path "/22e05ee1-b227-4be7-9418-94433f274720/00000000-0000-0000-0000-00005f5829d3"
-          (reference "#PWR01106") (unit 1)
+          (reference "#PWR?") (unit 1)
+        )
+      )
+      (project "LED_Panel_Controller"
+        (path "/22e05ee1-b227-4be7-9418-94433f274720/00000000-0000-0000-0000-00005f5829d3"
+          (reference "#PWR?") (unit 1)
         )
       )
@@
   (symbol (lib_id "Custom_Library:GNDA_MZ") (at 113.03 158.496 0) (unit 1)
     (in_bom yes) (on_board yes) (dnp no)
-    (property "Reference" "#PWR01008" (at 113.03 164.846 0)
+    (property "Reference" "#PWR?" (at 113.03 164.846 0)
       (effects (font (size 1.27 1.27)) hide)
     )
@@
       (project "Nixie_Clock_Core"
         (path "/16fdce21-b570-4d81-a458-e8839d611806/f7cc5c4d-c1a6-4096-b212-cb6ae1584770"
-          (reference "#PWR01008") (unit 1)
-        )
-      )
-      (project "LED_Panel_Controller"
-        (path "/22e05ee1-b227-4be7-9418-94433f274720/00000000-0000-0000-0000-00005f5829d3"
-          (reference "#PWR01103") (unit 1)
+          (reference "#PWR?") (unit 1)
+        )
+      )
+      (project "LED_Panel_Controller"
+        (path "/22e05ee1-b227-4be7-9418-94433f274720/00000000-0000-0000-0000-00005f5829d3"
+          (reference "#PWR?") (unit 1)
         )
       )
@@
   (symbol (lib_id "Custom_Library:PIC32MZ2048EFG100_IPF") (at 129.54 90.424 0) (unit 1)
     (in_bom yes) (on_board yes) (dnp no)
-    (property "Reference" "U1002" (at 175.26 153.924 0)
+    (property "Reference" "U?" (at 175.26 153.924 0)
       (effects (font (size 1.27 1.27)) (justify right))
     )
@@
       (project "Nixie_Clock_Core"
         (path "/16fdce21-b570-4d81-a458-e8839d611806/f7cc5c4d-c1a6-4096-b212-cb6ae1584770"
-          (reference "U1002") (unit 1)
-        )
-      )
-      (project "LED_Panel_Controller"
-        (path "/22e05ee1-b227-4be7-9418-94433f274720/00000000-0000-0000-0000-00005f5829d3"
-          (reference "U1101") (unit 1)
+          (reference "U?") (unit 1)
+        )
+      )
+      (project "LED_Panel_Controller"
+        (path "/22e05ee1-b227-4be7-9418-94433f274720/00000000-0000-0000-0000-00005f5829d3"
+          (reference "U?") (unit 1)
         )
       )
@@
   (symbol (lib_id "power:GND") (at 129.54 158.496 0) (unit 1)
     (in_bom yes) (on_board yes) (dnp no)
-    (property "Reference" "#PWR01010" (at 129.54 164.846 0)
+    (property "Reference" "#PWR?" (at 129.54 164.846 0)
       (effects (font (size 1.27 1.27)) hide)
     )
@@
       (project "Nixie_Clock_Core"
         (path "/16fdce21-b570-4d81-a458-e8839d611806/f7cc5c4d-c1a6-4096-b212-cb6ae1584770"
-          (reference "#PWR01010") (unit 1)
-        )
-      )
-      (project "LED_Panel_Controller"
-        (path "/22e05ee1-b227-4be7-9418-94433f274720/00000000-0000-0000-0000-00005f5829d3"
-          (reference "#PWR01105") (unit 1)
+          (reference "#PWR?") (unit 1)
+        )
+      )
+      (project "LED_Panel_Controller"
+        (path "/22e05ee1-b227-4be7-9418-94433f274720/00000000-0000-0000-0000-00005f5829d3"
+          (reference "#PWR?") (unit 1)
         )
       )
@@
   (symbol (lib_id "power:GND") (at 75.946 139.446 0) (unit 1)
     (in_bom yes) (on_board yes) (dnp no)
-    (property "Reference" "#PWR01004" (at 75.946 145.796 0)
+    (property "Reference" "#PWR?" (at 75.946 145.796 0)
       (effects (font (size 1.27 1.27)) hide)
     )
@@
       (project "Nixie_Clock_Core"
         (path "/16fdce21-b570-4d81-a458-e8839d611806/f7cc5c4d-c1a6-4096-b212-cb6ae1584770"
-          (reference "#PWR01004") (unit 1)
-        )
-      )
-      (project "LED_Panel_Controller"
-        (path "/22e05ee1-b227-4be7-9418-94433f274720/00000000-0000-0000-0000-00005f5829d3"
-          (reference "#PWR01101") (unit 1)
-        )
-      )
+          (reference "#PWR?") (unit 1)
+        )
+      )
+      (project "LED_Panel_Controller"
+        (path "/22e05ee1-b227-4be7-9418-94433f274720/00000000-0000-0000-0000-00005f5829d3"
+          (reference "#PWR?") (unit 1)
+        )
+      )

Commit message: more carrier board progress
Changed lines of the file:
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@@
+    )
+  )
+  (global_label "Anode_1" (shape input) (at 241.3 27.94 180)
+    (effects (font (size 1.27 1.27)) (justify right))
+    (property "Intersheetrefs" "${INTERSHEET_REFS}" (at 241.3 27.94 0)
+      (effects (font (size 1.27 1.27)) hide)
+    )
+  )
+  (global_label "Pushbutton_4" (shape output) (at 33.02 40.64 180) (fields_autoplaced)
+    (effects (font (size 1.27 1.27)) (justify right))
+    (property "Intersheetrefs" "${INTERSHEET_REFS}" (at 17.2936 40.64 0)
+      (effects (font (size 1.27 1.27)) (justify right) hide)
+    )
+  )
+  (global_label "Anode_5" (shape input) (at 241.3 38.1 180)
+    (effects (font (size 1.27 1.27)) (justify right))
+    (property "Intersheetrefs" "${INTERSHEET_REFS}" (at 241.3 38.1 0)
+      (effects (font (size 1.27 1.27)) hide)
     )
   )
@@
     (effects (font (size 1.27 1.27)) (justify right))
     (property "Intersheetrefs" "${INTERSHEET_REFS}" (at 78.74 124.714 0)
+      (effects (font (size 1.27 1.27)) hide)
+    )
+  )
+  (global_label "Anode_4" (shape input) (at 241.3 35.56 180)
+    (effects (font (size 1.27 1.27)) (justify right))
+    (property "Intersheetrefs" "${INTERSHEET_REFS}" (at 241.3 35.56 0)
+      (effects (font (size 1.27 1.27)) hide)
+    )
+  )
+  (global_label "Pushbutton_6" (shape output) (at 33.02 45.72 180) (fields_autoplaced)
+    (effects (font (size 1.27 1.27)) (justify right))
+    (property "Intersheetrefs" "${INTERSHEET_REFS}" (at 17.2936 45.72 0)
+      (effects (font (size 1.27 1.27)) (justify right) hide)
+    )
+  )
+  (global_label "~{Display_Detect}" (shape output) (at 33.02 48.26 180)
+    (effects (font (size 1.016 1.016)) (justify right))
+    (property "Intersheetrefs" "${INTERSHEET_REFS}" (at 33.02 48.26 0)
       (effects (font (size 1.27 1.27)) hide)
     )
@@
     )
   )
+  (global_label "Colon_1" (shape input) (at 241.3 71.12 180)
+    (effects (font (size 1.27 1.27)) (justify right))
+    (property "Intersheetrefs" "${INTERSHEET_REFS}" (at 241.3 71.12 0)
+      (effects (font (size 1.27 1.27)) hide)
+    )
+  )
+  (global_label "Anode_8" (shape input) (at 241.3 60.96 180)
+    (effects (font (size 1.27 1.27)) (justify right))
+    (property "Intersheetrefs" "${INTERSHEET_REFS}" (at 241.3 60.96 0)
+      (effects (font (size 1.27 1.27)) hide)
+    )
+  )
   (global_label "PIC32MZ_REFCLK1" (shape output) (at 78.74 122.174 180)
     (effects (font (size 1.27 1.27)) (justify right))
     (property "Intersheetrefs" "${INTERSHEET_REFS}" (at 78.74 122.174 0)
+      (effects (font (size 1.27 1.27)) hide)
+    )
+  )
+  (global_label "Anode_7" (shape input) (at 241.3 43.18 180)
+    (effects (font (size 1.27 1.27)) (justify right))
+    (property "Intersheetrefs" "${INTERSHEET_REFS}" (at 241.3 43.18 0)
       (effects (font (size 1.27 1.27)) hide)
     )
@@
     )
   )
+  (global_label "~{IO_Level_Shift_Enable}" (shape input) (at 233.68 48.26 180)
+    (effects (font (size 1.016 1.016)) (justify right))
+    (property "Intersheetrefs" "${INTERSHEET_REFS}" (at 233.68 48.26 0)
+      (effects (font (size 1.27 1.27)) hide)
+    )
+  )
+  (global_label "Anode_3" (shape input) (at 241.3 33.02 180)
+    (effects (font (size 1.27 1.27)) (justify right))
+    (property "Intersheetrefs" "${INTERSHEET_REFS}" (at 241.3 33.02 0)
+      (effects (font (size 1.27 1.27)) hide)
+    )
+  )
   (global_label "~{ETC_Config}" (shape input) (at 78.74 51.054 180)
     (effects (font (size 1.016 1.016)) (justify right))
     (property "Intersheetrefs" "${INTERSHEET_REFS}" (at 78.74 51.054 0)
+      (effects (font (size 1.27 1.27)) hide)
+    )
+  )
+  (global_label "Colon_2" (shape input) (at 241.3 73.66 180)
+    (effects (font (size 1.27 1.27)) (justify right))
+    (property "Intersheetrefs" "${INTERSHEET_REFS}" (at 241.3 73.66 0)
+      (effects (font (size 1.27 1.27)) hide)
+    )
+  )
+  (global_label "Pushbutton_1" (shape output) (at 33.02 33.02 180) (fields_autoplaced)
+    (effects (font (size 1.27 1.27)) (justify right))
+    (property "Intersheetrefs" "${INTERSHEET_REFS}" (at 17.2936 33.02 0)
+      (effects (font (size 1.27 1.27)) (justify right) hide)
+    )
+  )
+  (global_label "Anode_6" (shape input) (at 241.3 40.64 180)
+    (effects (font (size 1.27 1.27)) (justify right))
+    (property "Intersheetrefs" "${INTERSHEET_REFS}" (at 241.3 40.64 0)
       (effects (font (size 1.27 1.27)) hide)
     )
@@
     )
   )
+  (global_label "Pushbutton_5" (shape output) (at 33.02 43.18 180) (fields_autoplaced)
+    (effects (font (size 1.27 1.27)) (justify right))
+    (property "Intersheetrefs" "${INTERSHEET_REFS}" (at 17.2936 43.18 0)
+      (effects (font (size 1.27 1.27)) (justify right) hide)
+    )
+  )
+  (global_label "Pushbutton_0" (shape output) (at 33.02 30.48 180) (fields_autoplaced)
+    (effects (font (size 1.27 1.27)) (justify right))
+    (property "Intersheetrefs" "${INTERSHEET_REFS}" (at 17.2936 30.48 0)
+      (effects (font (size 1.27 1.27)) (justify right) hide)
+    )
+  )
+  (global_label "Pushbutton_2" (shape output) (at 33.02 35.56 180) (fields_autoplaced)
+    (effects (font (size 1.27 1.27)) (justify right))
+    (property "Intersheetrefs" "${INTERSHEET_REFS}" (at 17.2936 35.56 0)
+      (effects (font (size 1.27 1.27)) (justify right) hide)
+    )
+  )
+  (global_label "Colon_3" (shape input) (at 241.3 76.2 180)
+    (effects (font (size 1.27 1.27)) (justify right))
+    (property "Intersheetrefs" "${INTERSHEET_REFS}" (at 241.3 76.2 0)
+      (effects (font (size 1.27 1.27)) hide)
+    )
+  )
+  (global_label "Colon_0" (shape input) (at 241.3 68.58 180)
+    (effects (font (size 1.27 1.27)) (justify right))
+    (property "Intersheetrefs" "${INTERSHEET_REFS}" (at 241.3 68.58 0)
+      (effects (font (size 1.27 1.27)) hide)
+    )
+  )
+  (global_label "Pushbutton_3" (shape output) (at 33.02 38.1 180) (fields_autoplaced)
+    (effects (font (size 1.27 1.27)) (justify right))
+    (property "Intersheetrefs" "${INTERSHEET_REFS}" (at 17.2936 38.1 0)
+      (effects (font (size 1.27 1.27)) (justify right) hide)
+    )
+  )
   (global_label "I2C_SCL" (shape output) (at 233.934 112.014 0)
     (effects (font (size 1.27 1.27)) (justify left))
@@
       (effects (font (size 1.27 1.27)) hide)
     )
+  )
+  (global_label "Anode_2" (shape input) (at 241.3 30.48 180)
+    (effects (font (size 1.27 1.27)) (justify right))
+    (property "Intersheetrefs" "${INTERSHEET_REFS}" (at 241.3 30.48 0)
+      (effects (font (size 1.27 1.27)) hide)
+    )
+  )
+  (global_label "Anode_0" (shape input) (at 241.3 25.4 180)
+    (effects (font (size 1.27 1.27)) (justify right))
+    (property "Intersheetrefs" "${INTERSHEET_REFS}" (at 241.3 25.4 0)
+      (effects (font (size 1.27 1.27)) hide)
+    )
+  )
+  (global_label "Anode_DP" (shape input) (at 241.3 66.04 180)
+    (effects (font (size 1.27 1.27)) (justify right))
+    (property "Intersheetrefs" "${INTERSHEET_REFS}" (at 241.3 66.04 0)
+      (effects (font (size 1.27 1.27)) hide)
+    )
+  )
+  (global_label "Anode_9" (shape input) (at 241.3 63.5 180)
+    (effects (font (size 1.27 1.27)) (justify right))
+    (property "Intersheetrefs" "${INTERSHEET_REFS}" (at 241.3 63.5 0)
+      (effects (font (size 1.27 1.27)) hide)
+    )
