File: rev_b/hdw/Nixie_Clock_Core/USB_UART_Bridge.kicad_sch (KiCad schematic)
At the start: 37 parts, among them U1303 74LVC1G97, U1304 ISO7321C

Commit message: added BOM
Parts:
- L? (x2): Digi-Key PN (none) -> 490-1014-1-ND
- R? (x4): Digi-Key PN (none) -> 541-100KHCT-ND
- R? (x2): Digi-Key PN (none) -> 541-5306-1-ND
- R?: Digi-Key PN (none) -> 541-487KHCT-ND
- R?: Digi-Key PN (none) -> 541-10.0KHCT-ND
- R?: Digi-Key PN (none) -> 541-5412-1-ND
- R? (x2): Digi-Key PN (none) -> 541-1.00KHCT-ND
- R?: Digi-Key PN (none) -> 541-CRCW06036K04FKEBCT-ND
- U1303: Digi-Key PN (none) -> 296-15582-1-ND
- U1304: Digi-Key PN (none) -> 296-42102-1-ND
Other:
- title: (none) -> Nixie Clock Redux Core Board
Changed lines of the file:
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@@
   (paper "A")
   (title_block
-    (date "2023-05-12")
-    (rev "PRELIM")
+    (title "Nixie Clock Redux Core Board")
+    (date "2023-07-30")
+    (rev "B")
     (company "Drew Maatman")
   )
@@
     (effects (font (size 1.27 1.27)) (justify left bottom))
   )
-  (global_label "USB_UART_TX_ISO" (shape output) (at 208.28 36.83 0)
+  (global_label "USB_UART_TX_ISO" (shape output) (at 208.28 36.83 0) (fields_autoplaced)
     (effects (font (size 1.27 1.27)) (justify left))
-    (property "Intersheetrefs" "${INTERSHEET_REFS}" (at 208.28 36.83 0)
-      (effects (font (size 1.27 1.27)) hide)
-    )
-  )
-  (global_label "USB_UART_TX" (shape input) (at 60.96 36.83 180)
+    (property "Intersheetrefs" "${INTERSHEET_REFS}" (at 227.8772 36.83 0)
+      (effects (font (size 1.27 1.27)) (justify left))
+    )
+  )
+  (global_label "USB_UART_TX" (shape input) (at 60.96 36.83 180) (fields_autoplaced)
     (effects (font (size 1.27 1.27)) (justify right))
-    (property "Intersheetrefs" "${INTERSHEET_REFS}" (at 60.96 36.83 0)
-      (effects (font (size 1.27 1.27)) hide)
-    )
-  )
-  (global_label "~{USB_ACTIVE}" (shape passive) (at 95.25 114.3 0)
+    (property "Intersheetrefs" "${INTERSHEET_REFS}" (at 45.4752 36.83 0)
+      (effects (font (size 1.27 1.27)) (justify right))
+    )
+  )
+  (global_label "~{USB_ACTIVE}" (shape passive) (at 95.25 114.3 0) (fields_autoplaced)
     (effects (font (size 1.27 1.27)) (justify left))
-    (property "Intersheetrefs" "${INTERSHEET_REFS}" (at 95.25 114.3 0)
-      (effects (font (size 1.27 1.27)) hide)
-    )
-  )
-  (global_label "USB_UART_RX_ISO" (shape input) (at 208.28 34.29 0)
+    (property "Intersheetrefs" "${INTERSHEET_REFS}" (at 107.9907 114.3 0)
+      (effects (font (size 1.27 1.27)) (justify left))
+    )
+  )
+  (global_label "USB_UART_RX_ISO" (shape input) (at 208.28 34.29 0) (fields_autoplaced)
     (effects (font (size 1.27 1.27)) (justify left))
-    (property "Intersheetrefs" "${INTERSHEET_REFS}" (at 208.28 34.29 0)
-      (effects (font (size 1.27 1.27)) hide)
-    )
-  )
-  (global_label "USB_UART_RX" (shape output) (at 60.96 34.29 180)
+    (property "Intersheetrefs" "${INTERSHEET_REFS}" (at 228.1796 34.29 0)
+      (effects (font (size 1.27 1.27)) (justify left))
+    )
+  )
+  (global_label "USB_UART_RX" (shape output) (at 60.96 34.29 180) (fields_autoplaced)
     (effects (font (size 1.27 1.27)) (justify right))
-    (property "Intersheetrefs" "${INTERSHEET_REFS}" (at 60.96 34.29 0)
-      (effects (font (size 1.27 1.27)) hide)
-    )
-  )
-  (global_label "POS5_USB_PGOOD" (shape output) (at 74.93 154.94 0)
+    (property "Intersheetrefs" "${INTERSHEET_REFS}" (at 45.1728 34.29 0)
+      (effects (font (size 1.27 1.27)) (justify right))
+    )
+  )
+  (global_label "POS5_USB_PGOOD" (shape output) (at 74.93 154.94 0) (fields_autoplaced)
     (effects (font (size 1.27 1.27)) (justify left))
-    (property "Intersheetrefs" "${INTERSHEET_REFS}" (at 74.93 154.94 0)
-      (effects (font (size 1.27 1.27)) hide)
-    )
-  )
-  (global_label "USB_UART_RX_ISO" (shape output) (at 62.23 101.6 180)
+    (property "Intersheetrefs" "${INTERSHEET_REFS}" (at 95.0715 154.94 0)
+      (effects (font (size 1.27 1.27)) (justify left))
+    )
+  )
+  (global_label "USB_UART_RX_ISO" (shape output) (at 62.23 101.6 180) (fields_autoplaced)
     (effects (font (size 1.27 1.27)) (justify right))
-    (property "Intersheetrefs" "${INTERSHEET_REFS}" (at 62.23 101.6 0)
-      (effects (font (size 1.27 1.27)) hide)
-    )
-  )
-  (global_label "~{USB_ACTIVE}" (shape passive) (at 25.4 111.76 270)
+    (property "Intersheetrefs" "${INTERSHEET_REFS}" (at 42.3304 101.6 0)
+      (effects (font (size 1.27 1.27)) (justify right))
+    )
+  )
+  (global_label "~{USB_ACTIVE}" (shape passive) (at 25.4 111.76 270) (fields_autoplaced)
     (effects (font (size 1.27 1.27)) (justify right))
-    (property "Intersheetrefs" "${INTERSHEET_REFS}" (at 25.4 111.76 0)
-      (effects (font (size 1.27 1.27)) hide)
-    )
-  )
-  (global_label "POS5_USB_PGOOD" (shape input) (at 114.3 171.45 180)
+    (property "Intersheetrefs" "${INTERSHEET_REFS}" (at 25.4 124.5007 90)
+      (effects (font (size 1.27 1.27)) (justify right))
+    )
+  )
+  (global_label "POS5_USB_PGOOD" (shape input) (at 114.3 171.45 180) (fields_autoplaced)
     (effects (font (size 1.27 1.27)) (justify right))
-    (property "Intersheetrefs" "${INTERSHEET_REFS}" (at 114.3 171.45 0)
-      (effects (font (size 1.27 1.27)) hide)
-    )
-  )
-  (global_label "USB_UART_TX_ISO" (shape input) (at 62.23 104.14 180)
+    (property "Intersheetrefs" "${INTERSHEET_REFS}" (at 94.1585 171.45 0)
+      (effects (font (size 1.27 1.27)) (justify right))
+    )
+  )
+  (global_label "USB_UART_TX_ISO" (shape input) (at 62.23 104.14 180) (fields_autoplaced)
     (effects (font (size 1.27 1.27)) (justify right))
-    (property "Intersheetrefs" "${INTERSHEET_REFS}" (at 62.23 104.14 0)
-      (effects (font (size 1.27 1.27)) hide)
+    (property "Intersheetrefs" "${INTERSHEET_REFS}" (at 42.6328 104.14 0)
+      (effects (font (size 1.27 1.27)) (justify right))
     )
   )
@@
       (effects (font (size 1.27 1.27)) (justify left))
     )
-    (property "Digi-Key PN" "" (at 181.61 27.94 0)
+    (property "Digi-Key PN" "541-100KHCT-ND" (at 181.61 27.94 0)
       (effects (font (size 1.27 1.27)) hide)
     )
@@
       (effects (font (size 1.27 1.27)) hide)
     )
-    (property "Digi-Key PN" "" (at 119.634 -106.426 0)
+    (property "Digi-Key PN" "490-1014-1-ND" (at 119.634 -106.426 0)
       (effects (font (size 1.27 1.27)) hide)
     )
@@
       (effects (font (size 1.27 1.27)))
     )
-    (property "Digi-Key PN" "" (at 142.24 116.84 0)
+    (property "Digi-Key PN" "541-5306-1-ND" (at 142.24 116.84 0)
       (effects (font (size 1.524 1.524)) hide)
     )
@@
       (effects (font (size 1.27 1.27)) (justify left))
     )
-    (property "Digi-Key PN" "" (at 34.29 137.16 0)
+    (property "Digi-Key PN" "541-487KHCT-ND" (at 34.29 137.16 0)
       (effects (font (size 1.524 1.524)) hide)
     )
@@
       (effects (font (size 1.27 1.27)))
     )
-    (property "Digi-Key PN" "" (at 142.24 99.06 0)
+    (property "Digi-Key PN" "541-5306-1-ND" (at 142.24 99.06 0)
       (effects (font (size 1.524 1.524)) hide)
     )
@@
       (effects (font (size 1.27 1.27)) (justify left))
     )
-    (property "Digi-Key PN" "" (at 74.93 135.89 0)
+    (property "Digi-Key PN" "541-10.0KHCT-ND" (at 74.93 135.89 0)
       (effects (font (size 1.524 1.524)) hide)
     )
@@
       (effects (font (size 1.27 1.27)) hide)
     )
-    (property "Digi-Key PN" "" (at 136.906 -123.952 0)
+    (property "Digi-Key PN" "490-1014-1-ND" (at 136.906 -123.952 0)
       (effects (font (size 1.27 1.27)) hide)
     )
@@
       (effects (font (size 1.27 1.27)) (justify left))
     )
-    (property "Digi-Key PN" "" (at 194.31 27.94 0)
+    (property "Digi-Key PN" "541-100KHCT-ND" (at 194.31 27.94 0)
       (effects (font (size 1.27 1.27)) hide)
     )
@@
       (effects (font (size 1.27 1.27)) (justify left))
     )
-    (property "Digi-Key PN" "" (at 34.29 163.83 0)
+    (property "Digi-Key PN" "541-5412-1-ND" (at 34.29 163.83 0)
       (effects (font (size 1.524 1.524)) hide)
     )
@@
       (effects (font (size 1.27 1.27)) (justify left))
     )
-    (property "Digi-Key PN" "" (at 33.02 90.17 0)
+    (property "Digi-Key PN" "541-1.00KHCT-ND" (at 33.02 90.17 0)
       (effects (font (size 1.524 1.524)) hide)
     )
@@
       (effects (font (size 1.27 1.27)) (justify left))
     )
-    (property "Digi-Key PN" "" (at 73.66 27.94 0)
+    (property "Digi-Key PN" "541-100KHCT-ND" (at 73.66 27.94 0)
       (effects (font (size 1.27 1.27)) hide)
     )
@@
       (effects (font (size 1.27 1.27)) (justify left))
     )
-    (property "Digi-Key PN" "" (at 34.29 151.13 0)
+    (property "Digi-Key PN" "541-CRCW06036K04FKEBCT-ND" (at 34.29 151.13 0)
       (effects (font (size 1.524 1.524)) hide)
     )
@@
       (effects (font (size 1.27 1.27)) hide)
     )
+    (property "Digi-Key PN" "296-15582-1-ND" (at 121.92 171.45 0)
+      (effects (font (size 1.27 1.27)) hide)
+    )
     (pin "1")
     (pin "2")
@@
       (effects (font (size 1.27 1.27)) (justify left))
     )
-    (property "Digi-Key PN" "" (at 128.27 147.32 0)
+    (property "Digi-Key PN" "541-1.00KHCT-ND" (at 128.27 147.32 0)
       (effects (font (size 1.524 1.524)) hide)
     )
@@
     )
     (property "Datasheet" "http://www.ti.com/general/docs/lit/getliterature.tsp?genericPartNumber=iso7321c&fileType=pdf" (at 134.62 31.75 0)
+      (effects (font (size 1.27 1.27)) hide)
+    )
+    (property "Digi-Key PN" "296-42102-1-ND" (at 134.62 31.75 0)
       (effects (font (size 1.27 1.27)) hide)
     )
@@
       (effects (font (size 1.27 1.27)) (justify left))
     )
-    (property "Digi-Key PN" "" (at 86.36 27.94 0)
-      (effects (font (size 1.27 1.27)) hide)
-    )
+    (property "Digi-Key PN" "541-100KHCT-ND" (at 86.36 27.94 0)
+      (effects (font (size 1.27 1.27)) hide)
+    )
