File: rev_b/hdw/Nixie_Clock_Core/IO Connectors.kicad_sch (KiCad schematic)
At the start: 4 parts, among them J1901 Conn_02x32_Top_Bottom

Commit message: added BOM
Parts:
- C? (x2): Digi-Key PN (none) -> 565-4697-1-ND
Other:
- title: (none) -> Nixie Clock Redux Core Board
