File: rev_b/hdw/Nixie_Clock_Core/power_input.kicad_sch (KiCad schematic)
At the start: 24 parts

Commit message: added BOM
Parts:
- C?: Digi-Key PN (none) -> 399-16639-1-ND
- R? (x6): Digi-Key PN (none) -> 541-10.0KHCT-ND
- R? (x2): Digi-Key PN (none) -> 541-10.0HCT-ND
- R?: Digi-Key PN (none) -> 541-5237-1-ND
- R?: Digi-Key PN (none) -> 541-4027-1-ND
- R?: Digi-Key PN (none) -> 541-1.78KHCT-ND
Other:
- title: (none) -> Nixie Clock Redux Core Board
Changed lines of the file:
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@@
   (paper "A")
   (title_block
-    (date "2023-05-12")
-    (rev "PRELIM")
+    (title "Nixie Clock Redux Core Board")
+    (date "2023-07-30")
+    (rev "B")
     (company "Drew Maatman")
   )
@@
     (effects (font (size 1.27 1.27)) (justify left bottom))
   )
-  (global_label "POS24_SNS+" (shape passive) (at 165.1 44.45 90)
+  (global_label "POS24_SNS+" (shape passive) (at 165.1 44.45 90) (fields_autoplaced)
     (effects (font (size 1.27 1.27)) (justify left))
-    (property "Intersheetrefs" "${INTERSHEET_REFS}" (at 165.1 44.45 0)
-      (effects (font (size 1.27 1.27)) hide)
-    )
-  )
-  (global_label "POS24_SNS-" (shape passive) (at 177.8 44.45 90)
+    (property "Intersheetrefs" "${INTERSHEET_REFS}" (at 165.1 30.137 90)
+      (effects (font (size 1.27 1.27)) (justify left))
+    )
+  )
+  (global_label "POS24_SNS-" (shape passive) (at 177.8 44.45 90) (fields_autoplaced)
     (effects (font (size 1.27 1.27)) (justify left))
-    (property "Intersheetrefs" "${INTERSHEET_REFS}" (at 177.8 44.45 0)
-      (effects (font (size 1.27 1.27)) hide)
-    )
-  )
-  (global_label "POS24_PGOOD" (shape output) (at 220.98 105.41 0)
+    (property "Intersheetrefs" "${INTERSHEET_REFS}" (at 177.8 30.137 90)
+      (effects (font (size 1.27 1.27)) (justify left))
+    )
+  )
+  (global_label "POS24_PGOOD" (shape output) (at 220.98 105.41 0) (fields_autoplaced)
     (effects (font (size 1.27 1.27)) (justify left))
-    (property "Intersheetrefs" "${INTERSHEET_REFS}" (at 220.98 105.41 0)
-      (effects (font (size 1.27 1.27)) hide)
+    (property "Intersheetrefs" "${INTERSHEET_REFS}" (at 237.5534 105.41 0)
+      (effects (font (size 1.27 1.27)) (justify left))
     )
   )
@@
       (effects (font (size 1.27 1.27)) (justify left))
     )
-    (property "Digi-Key PN" "" (at 179.07 121.92 0)
+    (property "Digi-Key PN" "541-10.0KHCT-ND" (at 179.07 121.92 0)
       (effects (font (size 1.524 1.524)) hide)
     )
@@
       (effects (font (size 1.27 1.27)) hide)
     )
-    (property "Digi-Key PN" "" (at 165.1 48.26 0)
+    (property "Digi-Key PN" "541-10.0HCT-ND" (at 165.1 48.26 0)
       (effects (font (size 1.27 1.27)) hide)
     )
@@
       (effects (font (size 1.27 1.27)) (justify left))
     )
-    (property "Digi-Key PN" "" (at 194.31 121.92 0)
+    (property "Digi-Key PN" "541-10.0KHCT-ND" (at 194.31 121.92 0)
       (effects (font (size 1.524 1.524)) hide)
     )
@@
       (effects (font (size 1.27 1.27)) (justify left))
     )
-    (property "Digi-Key PN" "" (at 210.82 101.6 0)
+    (property "Digi-Key PN" "541-5237-1-ND" (at 210.82 101.6 0)
       (effects (font (size 1.524 1.524)) hide)
     )
@@
       (effects (font (size 1.27 1.27)) (justify left))
     )
-    (property "Digi-Key PN" "" (at 210.82 88.9 0)
+    (property "Digi-Key PN" "541-10.0KHCT-ND" (at 210.82 88.9 0)
       (effects (font (size 1.524 1.524)) hide)
     )
@@
       (effects (font (size 1.27 1.27)) (justify left))
     )
-    (property "Digi-Key PN" "" (at 109.22 57.15 0)
+    (property "Digi-Key PN" "541-4027-1-ND" (at 109.22 57.15 0)
       (effects (font (size 1.524 1.524)) hide)
     )
@@
       (effects (font (size 1.27 1.27)) (justify left))
     )
-    (property "Digi-Key PN" "" (at 210.82 121.92 0)
+    (property "Digi-Key PN" "541-10.0KHCT-ND" (at 210.82 121.92 0)
       (effects (font (size 1.524 1.524)) hide)
     )
@@
       (effects (font (size 1.27 1.27)) (justify left))
     )
-    (property "Digi-Key PN" "" (at 114.3 57.15 0)
+    (property "Digi-Key PN" "541-10.0KHCT-ND" (at 114.3 57.15 0)
       (effects (font (size 1.524 1.524)) hide)
     )
@@
       (effects (font (size 1.27 1.27)) (justify left))
     )
-    (property "Digi-Key PN" "" (at 109.22 80.01 0)
+    (property "Digi-Key PN" "541-1.78KHCT-ND" (at 109.22 80.01 0)
       (effects (font (size 1.524 1.524)) hide)
     )
@@
       (effects (font (size 1.27 1.27)) (justify left))
     )
-    (property "Digi-Key PN" "" (at 109.22 101.6 0)
+    (property "Digi-Key PN" "541-10.0KHCT-ND" (at 109.22 101.6 0)
       (effects (font (size 1.524 1.524)) hide)
     )
@@
       (effects (font (size 1.27 1.27)) hide)
     )
-    (property "Digi-Key PN" "" (at 245.11 63.5 0)
+    (property "Digi-Key PN" "399-16639-1-ND" (at 245.11 63.5 0)
       (effects (font (size 1.27 1.27)) hide)
     )
@@
       (effects (font (size 1.27 1.27)) hide)
     )
-    (property "Digi-Key PN" "" (at 177.8 48.26 0)
-      (effects (font (size 1.27 1.27)) hide)
-    )
+    (property "Digi-Key PN" "541-10.0HCT-ND" (at 177.8 48.26 0)
+      (effects (font (size 1.27 1.27)) hide)
+    )

Commit message: regenerated production boms
Parts:
- added N201: 24V PSU, symbol Mechanical:Housing
Changed lines of the file:
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@@
   (title_block
     (title "Nixie Clock Redux Core Board")
-    (date "2023-08-11")
+    (date "2023-12-25")
     (rev "B")
     (company "Drew Maatman")
@@
         )
       )
+    )
+  )
+  (symbol (lib_id "Mechanical:Housing") (at 31.75 89.535 0) (unit 1)
+    (in_bom yes) (on_board yes) (dnp no)
+    (property "Reference" "N201" (at 35.56 89.535 0)
+      (effects (font (size 1.27 1.27)) (justify left))
+    )
+    (property "Value" "24V PSU" (at 35.56 91.44 0)
+      (effects (font (size 1.27 1.27)) (justify left))
+    )
+    (property "Footprint" "" (at 33.02 88.265 0)
+      (effects (font (size 1.27 1.27)) hide)
+    )
+    (property "Datasheet" "~" (at 33.02 88.265 0)
+      (effects (font (size 1.27 1.27)) hide)
+    )
+    (property "Digi-Key PN" "1939-1835-ND" (at 31.75 89.535 0)
+      (effects (font (size 1.27 1.27)) hide)
+    )
+    (instances
+      (project "Nixie_Clock_Core"
+        (path "/16fdce21-b570-4d81-a458-e8839d611806/033277b9-3b61-4d88-889d-97b223ca74c5"
+          (reference "N201") (unit 1)
+        )
+      )
