File: rev_b/hdw/IN12_carrier/IN12_carrier/Anode_Drive.kicad_sch (KiCad schematic)
At the start: 36 parts, among them Q1001 MMSTA92, Q1002 MMSTA92, Q1003 MMSTA42, Q1004 MMSTA42, Q1005 MMSTA92, Q1006 MMSTA92, Q1007 MMSTA42, Q1008 MMSTA42, Q1009 MMSTA92, Q1010 MMSTA92, Q1011 MMSTA42, Q1012 MMSTA42

Commit message: assigned digikey pns to IN12 carrier board parts
Parts:
- Q1001, Q1002, Q1005, Q1006, Q1009, Q1010: Digi-Key PN (none) -> MMSTA92-TPCT-ND
- Q1003, Q1004, Q1007, Q1008, Q1011, Q1012: Digi-Key PN (none) -> MMSTA42-FDICT-ND
- R401, R402, R403, R413, R414, R415: Digi-Key PN PN -> 541-10.0KHCT-ND
- R404, R405, R406, R416, R417, R418: Digi-Key PN PN -> 541-470KCCT-ND
- R407, R408, R409, R419, R420, R421: Digi-Key PN PN -> 541-4318-1-ND
- R410, R411, R412, R422, R423, R424: Digi-Key PN PN -> 541-18.0KCCT-ND
Changed lines of the file:
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@@
       (effects (font (size 1.27 1.27)))
     )
-    (property "Digi-Key PN" "PN" (at 151.13 82.55 0)
+    (property "Digi-Key PN" "541-470KCCT-ND" (at 151.13 82.55 0)
       (effects (font (size 1.524 1.524)) hide)
     )
@@
       (effects (font (size 1.27 1.27)))
     )
-    (property "Digi-Key PN" "PN" (at 151.13 129.54 0)
+    (property "Digi-Key PN" "541-470KCCT-ND" (at 151.13 129.54 0)
       (effects (font (size 1.524 1.524)) hide)
     )
@@
       (effects (font (size 1.27 1.27)) (justify left))
     )
-    (property "Digi-Key PN" "PN" (at 186.69 109.22 0)
+    (property "Digi-Key PN" "541-18.0KCCT-ND" (at 186.69 109.22 0)
       (effects (font (size 1.524 1.524)) hide)
     )
@@
       (effects (font (size 1.27 1.27)))
     )
-    (property "Digi-Key PN" "PN" (at 134.62 41.91 0)
+    (property "Digi-Key PN" "541-10.0KHCT-ND" (at 134.62 41.91 0)
       (effects (font (size 1.524 1.524)) hide)
     )
@@
       (effects (font (size 1.27 1.27)) (justify left))
     )
+    (property "Digi-Key PN" "MMSTA42-FDICT-ND" (at 153.67 97.79 0)
+      (effects (font (size 1.27 1.27)) hide)
+    )
     (pin "1")
     (pin "2")
@@
       (effects (font (size 1.27 1.27)) (justify left))
     )
+    (property "Digi-Key PN" "MMSTA92-TPCT-ND" (at 93.98 90.17 0)
+      (effects (font (size 1.27 1.27)) hide)
+    )
     (pin "1")
     (pin "2")
@@
       (effects (font (size 1.27 1.27)) (justify left))
     )
-    (property "Digi-Key PN" "PN" (at 104.14 156.21 0)
+    (property "Digi-Key PN" "541-18.0KCCT-ND" (at 104.14 156.21 0)
       (effects (font (size 1.524 1.524)) hide)
     )
@@
       (effects (font (size 1.27 1.27)))
     )
-    (property "Digi-Key PN" "PN" (at 52.07 90.17 0)
+    (property "Digi-Key PN" "541-10.0KHCT-ND" (at 52.07 90.17 0)
       (effects (font (size 1.524 1.524)) hide)
     )
@@
       (effects (font (size 1.27 1.27)) (justify left))
     )
+    (property "Digi-Key PN" "MMSTA92-TPCT-ND" (at 176.53 43.18 0)
+      (effects (font (size 1.27 1.27)) hide)
+    )
     (pin "1")
     (pin "2")
@@
       (effects (font (size 1.27 1.27)) (justify left))
     )
+    (property "Digi-Key PN" "MMSTA42-FDICT-ND" (at 71.12 49.53 0)
+      (effects (font (size 1.27 1.27)) hide)
+    )
     (pin "1")
     (pin "2")
@@
       (effects (font (size 1.27 1.27)))
     )
-    (property "Digi-Key PN" "PN" (at 134.62 137.16 0)
+    (property "Digi-Key PN" "541-10.0KHCT-ND" (at 134.62 137.16 0)
       (effects (font (size 1.524 1.524)) hide)
     )
@@
       (effects (font (size 1.27 1.27)))
     )
-    (property "Digi-Key PN" "PN" (at 151.13 35.56 0)
+    (property "Digi-Key PN" "541-470KCCT-ND" (at 151.13 35.56 0)
       (effects (font (size 1.524 1.524)) hide)
     )
@@
       (effects (font (size 1.27 1.27)))
     )
-    (property "Digi-Key PN" "PN" (at 162.56 26.67 0)
+    (property "Digi-Key PN" "541-4318-1-ND" (at 162.56 26.67 0)
       (effects (font (size 1.524 1.524)) hide)
     )
@@
       (effects (font (size 1.27 1.27)) (justify left))
     )
-    (property "Digi-Key PN" "PN" (at 104.14 109.22 0)
+    (property "Digi-Key PN" "541-18.0KCCT-ND" (at 104.14 109.22 0)
       (effects (font (size 1.524 1.524)) hide)
     )
@@
       (effects (font (size 1.27 1.27)) (justify left))
     )
+    (property "Digi-Key PN" "MMSTA42-FDICT-ND" (at 71.12 97.79 0)
+      (effects (font (size 1.27 1.27)) hide)
+    )
     (pin "1")
     (pin "2")
@@
       (effects (font (size 1.27 1.27)) (justify left))
     )
-    (property "Digi-Key PN" "PN" (at 186.69 156.21 0)
+    (property "Digi-Key PN" "541-18.0KCCT-ND" (at 186.69 156.21 0)
       (effects (font (size 1.524 1.524)) hide)
     )
@@
       (effects (font (size 1.27 1.27)))
     )
-    (property "Digi-Key PN" "PN" (at 68.58 129.54 0)
+    (property "Digi-Key PN" "541-470KCCT-ND" (at 68.58 129.54 0)
       (effects (font (size 1.524 1.524)) hide)
     )
@@
       (effects (font (size 1.27 1.27)) (justify left))
     )
-    (property "Digi-Key PN" "PN" (at 104.14 62.23 0)
+    (property "Digi-Key PN" "541-18.0KCCT-ND" (at 104.14 62.23 0)
       (effects (font (size 1.524 1.524)) hide)
     )
@@
       (effects (font (size 1.27 1.27)))
     )
-    (property "Digi-Key PN" "PN" (at 80.01 74.93 0)
+    (property "Digi-Key PN" "541-4318-1-ND" (at 80.01 74.93 0)
       (effects (font (size 1.524 1.524)) hide)
     )
@@
       (effects (font (size 1.27 1.27)))
     )
-    (property "Digi-Key PN" "PN" (at 162.56 74.93 0)
+    (property "Digi-Key PN" "541-4318-1-ND" (at 162.56 74.93 0)
       (effects (font (size 1.524 1.524)) hide)
     )
@@
       (effects (font (size 1.27 1.27)))
     )
-    (property "Digi-Key PN" "PN" (at 162.56 121.92 0)
+    (property "Digi-Key PN" "541-4318-1-ND" (at 162.56 121.92 0)
       (effects (font (size 1.524 1.524)) hide)
     )
@@
       (effects (font (size 1.27 1.27)))
     )
-    (property "Digi-Key PN" "PN" (at 80.01 26.67 0)
+    (property "Digi-Key PN" "541-4318-1-ND" (at 80.01 26.67 0)
       (effects (font (size 1.524 1.524)) hide)
     )
@@
       (effects (font (size 1.27 1.27)) (justify left))
     )
+    (property "Digi-Key PN" "MMSTA92-TPCT-ND" (at 176.53 137.16 0)
+      (effects (font (size 1.27 1.27)) hide)
+    )
     (pin "1")
     (pin "2")
@@
       (effects (font (size 1.27 1.27)) (justify left))
     )
+    (property "Digi-Key PN" "MMSTA42-FDICT-ND" (at 153.67 49.53 0)
+      (effects (font (size 1.27 1.27)) hide)
+    )
     (pin "1")
     (pin "2")
@@
       (effects (font (size 1.27 1.27)) (justify left))
     )
+    (property "Digi-Key PN" "MMSTA92-TPCT-ND" (at 93.98 43.18 0)
+      (effects (font (size 1.27 1.27)) hide)
+    )
     (pin "1")
     (pin "2")
@@
       (effects (font (size 1.27 1.27)))
     )
-    (property "Digi-Key PN" "PN" (at 52.07 137.16 0)
+    (property "Digi-Key PN" "541-10.0KHCT-ND" (at 52.07 137.16 0)
       (effects (font (size 1.524 1.524)) hide)
     )
@@
       (effects (font (size 1.27 1.27)) (justify left))
     )
+    (property "Digi-Key PN" "MMSTA42-FDICT-ND" (at 71.12 144.78 0)
+      (effects (font (size 1.27 1.27)) hide)
+    )
     (pin "1")
     (pin "2")
@@
       (effects (font (size 1.27 1.27)) (justify left))
     )
+    (property "Digi-Key PN" "MMSTA92-TPCT-ND" (at 176.53 90.17 0)
+      (effects (font (size 1.27 1.27)) hide)
+    )
     (pin "1")
     (pin "2")
@@
       (effects (font (size 1.27 1.27)))
     )
-    (property "Digi-Key PN" "PN" (at 68.58 82.55 0)
+    (property "Digi-Key PN" "541-470KCCT-ND" (at 68.58 82.55 0)
       (effects (font (size 1.524 1.524)) hide)
     )
@@
       (effects (font (size 1.27 1.27)) (justify left))
     )
-    (property "Digi-Key PN" "PN" (at 186.69 62.23 0)
+    (property "Digi-Key PN" "541-18.0KCCT-ND" (at 186.69 62.23 0)
       (effects (font (size 1.524 1.524)) hide)
     )
@@
       (effects (font (size 1.27 1.27)))
     )
-    (property "Digi-Key PN" "PN" (at 80.01 121.92 0)
+    (property "Digi-Key PN" "541-4318-1-ND" (at 80.01 121.92 0)
       (effects (font (size 1.524 1.524)) hide)
     )
@@
       (effects (font (size 1.27 1.27)))
     )
-    (property "Digi-Key PN" "PN" (at 134.62 90.17 0)
+    (property "Digi-Key PN" "541-10.0KHCT-ND" (at 134.62 90.17 0)
       (effects (font (size 1.524 1.524)) hide)
     )
@@
       (effects (font (size 1.27 1.27)) (justify left))
     )
+    (property "Digi-Key PN" "MMSTA92-TPCT-ND" (at 93.98 137.16 0)
+      (effects (font (size 1.27 1.27)) hide)
+    )
     (pin "1")
     (pin "2")
@@
       (effects (font (size 1.27 1.27)) (justify left))
     )
+    (property "Digi-Key PN" "MMSTA42-FDICT-ND" (at 153.67 144.78 0)
+      (effects (font (size 1.27 1.27)) hide)
+    )
     (pin "1")
     (pin "2")
@@
       (effects (font (size 1.27 1.27)))
     )
-    (property "Digi-Key PN" "PN" (at 68.58 35.56 0)
+    (property "Digi-Key PN" "541-470KCCT-ND" (at 68.58 35.56 0)
       (effects (font (size 1.524 1.524)) hide)
     )
@@
       (effects (font (size 1.27 1.27)))
     )
-    (property "Digi-Key PN" "PN" (at 52.07 41.91 0)
-      (effects (font (size 1.524 1.524)) hide)
-    )
+    (property "Digi-Key PN" "541-10.0KHCT-ND" (at 52.07 41.91 0)
+      (effects (font (size 1.524 1.524)) hide)
+    )
