File: rev_b/hdw/IN12_carrier/IN12_carrier/Cathode_Drive.kicad_sch (KiCad schematic)
At the start: 31 parts, among them Q901 MMSTA42, Q902 MMSTA42, Q904 MMSTA42, Q905 MMSTA42, Q906 MMSTA42, Q907 MMSTA42, Q908 MMSTA42, Q909 MMSTA42, Q910 MMSTA42, Q911 MMSTA42

Commit message: assigned digikey pns to IN12 carrier board parts
Parts:
- Q901, Q902, Q904, Q905, Q906, Q907, Q908, Q909, Q910, Q911: Digi-Key PN (none) -> MMSTA42-FDICT-ND
- R? (x15): Digi-Key PN PN -> 541-10.0KHCT-ND
- R?: Digi-Key PN PN -> 541-18.0KCCT-ND
Changed lines of the file:
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@@
       (effects (font (size 1.27 1.27)))
     )
-    (property "Digi-Key PN" "PN" (at 58.42 59.69 0)
+    (property "Digi-Key PN" "541-10.0KHCT-ND" (at 58.42 59.69 0)
       (effects (font (size 1.524 1.524)) hide)
     )
@@
       (effects (font (size 1.27 1.27)))
     )
-    (property "Digi-Key PN" "PN" (at 58.42 152.4 0)
+    (property "Digi-Key PN" "541-10.0KHCT-ND" (at 58.42 152.4 0)
       (effects (font (size 1.524 1.524)) hide)
     )
@@
       (effects (font (size 1.27 1.27)))
     )
-    (property "Digi-Key PN" "PN" (at 208.28 40.64 0)
+    (property "Digi-Key PN" "541-10.0KHCT-ND" (at 208.28 40.64 0)
       (effects (font (size 1.524 1.524)) hide)
     )
@@
       (effects (font (size 1.27 1.27)) (justify left))
     )
+    (property "Digi-Key PN" "MMSTA42-FDICT-ND" (at 77.47 160.02 0)
+      (effects (font (size 1.27 1.27)) hide)
+    )
     (pin "1")
     (pin "2")
@@
       (effects (font (size 1.27 1.27)) (justify left))
     )
+    (property "Digi-Key PN" "MMSTA42-FDICT-ND" (at 77.47 67.31 0)
+      (effects (font (size 1.27 1.27)) hide)
+    )
     (pin "1")
     (pin "2")
@@
       (effects (font (size 1.27 1.27)))
     )
-    (property "Digi-Key PN" "PN" (at 182.88 101.6 0)
+    (property "Digi-Key PN" "541-10.0KHCT-ND" (at 182.88 101.6 0)
       (effects (font (size 1.524 1.524)) hide)
     )
@@
       (effects (font (size 1.27 1.27)) (justify left))
     )
+    (property "Digi-Key PN" "MMSTA42-FDICT-ND" (at 152.4 128.27 0)
+      (effects (font (size 1.27 1.27)) hide)
+    )
     (pin "1")
     (pin "2")
@@
       (effects (font (size 1.27 1.27)))
     )
-    (property "Digi-Key PN" "PN" (at 133.35 152.4 0)
+    (property "Digi-Key PN" "541-10.0KHCT-ND" (at 133.35 152.4 0)
       (effects (font (size 1.524 1.524)) hide)
     )
@@
       (effects (font (size 1.27 1.27)))
     )
-    (property "Digi-Key PN" "PN" (at 182.88 137.16 0)
+    (property "Digi-Key PN" "541-10.0KHCT-ND" (at 182.88 137.16 0)
       (effects (font (size 1.524 1.524)) hide)
     )
@@
       (effects (font (size 1.27 1.27)) (justify left))
     )
+    (property "Digi-Key PN" "MMSTA42-FDICT-ND" (at 77.47 35.56 0)
+      (effects (font (size 1.27 1.27)) hide)
+    )
     (pin "1")
     (pin "2")
@@
       (effects (font (size 1.27 1.27)))
     )
-    (property "Digi-Key PN" "PN" (at 58.42 120.65 0)
+    (property "Digi-Key PN" "541-10.0KHCT-ND" (at 58.42 120.65 0)
       (effects (font (size 1.524 1.524)) hide)
     )
@@
       (effects (font (size 1.27 1.27)) (justify left))
     )
+    (property "Digi-Key PN" "MMSTA42-FDICT-ND" (at 152.4 160.02 0)
+      (effects (font (size 1.27 1.27)) hide)
+    )
     (pin "1")
     (pin "2")
@@
       (effects (font (size 1.27 1.27)) (justify left))
     )
+    (property "Digi-Key PN" "MMSTA42-FDICT-ND" (at 77.47 128.27 0)
+      (effects (font (size 1.27 1.27)) hide)
+    )
     (pin "1")
     (pin "2")
@@
       (effects (font (size 1.27 1.27)))
     )
-    (property "Digi-Key PN" "PN" (at 133.35 88.9 0)
+    (property "Digi-Key PN" "541-10.0KHCT-ND" (at 133.35 88.9 0)
       (effects (font (size 1.524 1.524)) hide)
     )
@@
       (effects (font (size 1.27 1.27)) (justify left))
     )
+    (property "Digi-Key PN" "MMSTA42-FDICT-ND" (at 77.47 96.52 0)
+      (effects (font (size 1.27 1.27)) hide)
+    )
     (pin "1")
     (pin "2")
@@
       (effects (font (size 1.27 1.27)) (justify left))
     )
+    (property "Digi-Key PN" "MMSTA42-FDICT-ND" (at 252.73 109.22 0)
+      (effects (font (size 1.27 1.27)) hide)
+    )
     (pin "1")
     (pin "2")
@@
       (effects (font (size 1.27 1.27)) (justify left))
     )
+    (property "Digi-Key PN" "MMSTA42-FDICT-ND" (at 252.73 144.78 0)
+      (effects (font (size 1.27 1.27)) hide)
+    )
     (pin "1")
     (pin "2")
@@
       (effects (font (size 1.27 1.27)))
     )
-    (property "Digi-Key PN" "PN" (at 58.42 27.94 0)
+    (property "Digi-Key PN" "541-10.0KHCT-ND" (at 58.42 27.94 0)
       (effects (font (size 1.524 1.524)) hide)
     )
@@
       (effects (font (size 1.27 1.27)))
     )
-    (property "Digi-Key PN" "PN" (at 233.68 101.6 0)
+    (property "Digi-Key PN" "541-10.0KHCT-ND" (at 233.68 101.6 0)
       (effects (font (size 1.524 1.524)) hide)
     )
@@
       (effects (font (size 1.27 1.27)) (justify left))
     )
+    (property "Digi-Key PN" "MMSTA42-FDICT-ND" (at 201.93 109.22 0)
+      (effects (font (size 1.27 1.27)) hide)
+    )
     (pin "1")
     (pin "2")
@@
       (effects (font (size 1.27 1.27)))
     )
-    (property "Digi-Key PN" "PN" (at 58.42 88.9 0)
+    (property "Digi-Key PN" "541-10.0KHCT-ND" (at 58.42 88.9 0)
       (effects (font (size 1.524 1.524)) hide)
     )
@@
       (effects (font (size 1.27 1.27)))
     )
-    (property "Digi-Key PN" "PN" (at 233.68 137.16 0)
+    (property "Digi-Key PN" "541-10.0KHCT-ND" (at 233.68 137.16 0)
       (effects (font (size 1.524 1.524)) hide)
     )
@@
       (effects (font (size 1.27 1.27)))
     )
-    (property "Digi-Key PN" "PN" (at 133.35 120.65 0)
+    (property "Digi-Key PN" "541-10.0KHCT-ND" (at 133.35 120.65 0)
       (effects (font (size 1.524 1.524)) hide)
     )
@@
       (effects (font (size 1.27 1.27)) (justify left))
     )
+    (property "Digi-Key PN" "MMSTA42-FDICT-ND" (at 152.4 35.56 0)
+      (effects (font (size 1.27 1.27)) hide)
+    )
     (pin "1")
     (pin "2")
@@
       (effects (font (size 1.27 1.27)) (justify left))
     )
+    (property "Digi-Key PN" "MMSTA42-FDICT-ND" (at 201.93 144.78 0)
+      (effects (font (size 1.27 1.27)) hide)
+    )
     (pin "1")
     (pin "2")
@@
       (effects (font (size 1.27 1.27)))
     )
-    (property "Digi-Key PN" "PN" (at 133.35 27.94 0)
+    (property "Digi-Key PN" "541-10.0KHCT-ND" (at 133.35 27.94 0)
       (effects (font (size 1.524 1.524)) hide)
     )
@@
       (effects (font (size 1.27 1.27)) (justify left))
     )
+    (property "Digi-Key PN" "MMSTA42-FDICT-ND" (at 152.4 67.31 0)
+      (effects (font (size 1.27 1.27)) hide)
+    )
     (pin "1")
     (pin "2")
@@
       (effects (font (size 1.27 1.27)) (justify left))
     )
+    (property "Digi-Key PN" "MMSTA42-FDICT-ND" (at 227.33 48.26 0)
+      (effects (font (size 1.27 1.27)) hide)
+    )
     (pin "1")
     (pin "2")
@@
       (effects (font (size 1.27 1.27)))
     )
-    (property "Digi-Key PN" "PN" (at 133.35 59.69 0)
+    (property "Digi-Key PN" "541-10.0KHCT-ND" (at 133.35 59.69 0)
       (effects (font (size 1.524 1.524)) hide)
     )
@@
       (effects (font (size 1.27 1.27)) (justify left))
     )
+    (property "Digi-Key PN" "MMSTA42-FDICT-ND" (at 152.4 96.52 0)
+      (effects (font (size 1.27 1.27)) hide)
+    )
     (pin "1")
     (pin "2")
@@
       (effects (font (size 1.27 1.27)) (justify left))
     )
-    (property "Digi-Key PN" "PN" (at 237.49 49.53 0)
+    (property "Digi-Key PN" "541-18.0KCCT-ND" (at 237.49 49.53 0)
       (effects (font (size 1.524 1.524)) hide)
     )
