File: rev_b/hdw/IN12_carrier/IN12_carrier/IN12_carrier.kicad_pcb (KiCad board)
At the start: 4 copper layers, 200 x 50 mm, 212 parts, among them J1001 Cap SNS, J201 Conn_02x32_Top_Bottom, Q401 MMSTA42, Q402 MMSTA42, Q403 MMSTA42, Q404 MMSTA92, Q405 MMSTA92, Q406 MMSTA92, Q407 MMSTA42, Q408 MMSTA42, Q409 MMSTA42, Q410 MMSTA92, Q411 MMSTA92, Q412 MMSTA92, Q501 MMSTA42, Q502 MMSTA42, Q503 MMSTA42, Q504 MMSTA42, Q505 MMSTA42, Q506 MMSTA42, Q507 MMSTA42, Q508 MMSTA42, Q509 MMSTA42, Q510 MMSTA42, Q511 MMSTA42, Q512 MMSTA42, Q513 MMSTA42, Q514 MMSTA42, Q515 MMSTA42, U1001 TCA9555RGER, U1002 24AA02-OT, U1003 AT42QT1010-TSHR, U1004 AT42QT1010-TSHR, U1005 AT42QT1010-TSHR, U1006 AT42QT1010-TSHR, U1007 AT42QT1010-TSHR, U301 DS1683, U302 LTC4316DD, U701 LP5009, U702 LP5009, U703 LP5009

Commit message: updated laser cut to add 1/8th inch margin on all sides, LED holes, wider tube gaps
Parts:
- added G***: N/A, LEDs:LED_0603, F.Cu at (141.7, 84.8)
- added G***: N/A, LEDs:LED_0603, F.Cu at (143.7, 84.8)
- added G***: N/A, LEDs:LED_0603, F.Cu at (135.3, 84.8)
- added G***: N/A, LEDs:LED_0603, F.Cu at (145.9, 84.8)
- added G***: N/A, LEDs:LED_0603, F.Cu at (126.9, 84.8)
- added G***: N/A, LEDs:LED_0603, F.Cu at (148.0, 84.8)
- added G***: N/A, LEDs:LED_0603, F.Cu at (137.5, 84.8)
- added G***: N/A, LEDs:LED_0603, F.Cu at (124.7, 84.8)
- added G***: N/A, LEDs:LED_0603, F.Cu at (133.2, 84.8)
- added G***: N/A, LEDs:LED_0603, F.Cu at (139.6, 84.8)
- added G***: N/A, LEDs:LED_0603, F.Cu at (131.0, 84.8)
- added G***: N/A, LEDs:LED_0603, F.Cu at (129.0, 84.8)
